Commit message: Fixed .stl references in lidar.xacro

File: urdf/lidar.xacro (robot description, xacro)
@@ -18,5 +18,5 @@
             <visual>
                 <geometry>
-                    <mesh filename="package://rotating_lidar_sensor/models/sensor_cylinder.stl"/>
+                    <mesh filename="package://rotating_lidar_sensor_position_controller/models/sensor_cylinder.stl"/>
                 </geometry>
                 <material name="grey"/>
@@ -24,5 +24,5 @@
             <collision>
                 <geometry>
-                    <mesh filename="package://rotating_lidar_sensor/models/sensor_cylinder.stl"/>
+                    <mesh filename="package://rotating_lidar_sensor_position_controller/models/sensor_cylinder.stl"/>
                 </geometry>
                 <surface>
@@ -52,5 +52,5 @@
             <visual>
                 <geometry>
-                    <mesh filename="package://rotating_lidar_sensor/models/sensor_plate.stl"/>
+                    <mesh filename="package://rotating_lidar_sensor_position_controller/models/sensor_plate.stl"/>
                 </geometry>
                 <material name="red"/>
@@ -58,5 +58,5 @@
             <collision>
                 <geometry>
-                    <mesh filename="package://rotating_lidar_sensor/models/sensor_plate.stl"/>
+                    <mesh filename="package://rotating_lidar_sensor_position_controller/models/sensor_plate.stl"/>
                 </geometry>
                 <surface>
@@ -86,5 +86,5 @@
             <visual>
                 <geometry>
-                    <mesh filename="package://rotating_lidar_sensor/models/Garmin_Lidar_Lite_3.stl"/>
+                    <mesh filename="package://rotating_lidar_sensor_position_controller/models/Garmin_Lidar_Lite_3.stl"/>
                 </geometry>
                 <material name="black"/>
@@ -92,5 +92,5 @@
             <collision>
                 <geometry>
-                    <mesh filename="package://rotating_lidar_sensor/models/Garmin_Lidar_Lite_3.stl"/>
+                    <mesh filename="package://rotating_lidar_sensor_position_controller/models/Garmin_Lidar_Lite_3.stl"/>
                 </geometry>
             </collision>

Commit message: Fixed Sensor mass and inertia values, adapted PID controller values

File: urdf/lidar.xacro (robot description, xacro)
@@ -13,8 +13,8 @@
         <!-- LIDAR SENSOR BASE LINK -->
         <link name="sensor_base_link">
-            <!--radius = 2mm heigth = 1mm-->
-            <xacro:property name="radius" value="0.20"/>
-            <xacro:property name="heigth" value="0.10"/>
-            <xacro:property name="mass" value="0.100"/>
+            <!--radius = 20mm heigth = 10mm-->
+            <xacro:property name="radius" value="0.02"/>
+            <xacro:property name="heigth" value="0.01"/>
+            <xacro:property name="mass" value="0.01"/>
             <visual>
                 <geometry>
@@ -46,9 +46,8 @@
         <!-- LIDAR SENSOR Mounting Plate LINK -->
         <link name="sensor_mounting_plate_link">
-            <!--radius = 2mm heigth = 0.1mm-->
-            <!-- values in cm and g-->
-            <xacro:property name="radius" value="0.20"/>
+            <!--radius = 20mm heigth = 1mm-->
+            <xacro:property name="radius" value="0.2"/>
             <xacro:property name="heigth" value="0.1"/>
-            <xacro:property name="mass" value="0.10"/>
+            <xacro:property name="mass" value="0.1"/>
             <visual>
                 <geometry>
@@ -81,8 +80,8 @@
         <link name="laser_frame">
             <!--length = 40mm, width = 48mm, heigth = 20mm, mass = 22g-->
-            <xacro:property name="length" value="0.40"/>
-            <xacro:property name="width" value="0.48"/>
-            <xacro:property name="heigth" value="0.20"/>
-            <xacro:property name="mass" value="0.22"/>
+            <xacro:property name="length" value="0.040"/>
+            <xacro:property name="width" value="0.048"/>
+            <xacro:property name="heigth" value="0.020"/>
+            <xacro:property name="mass" value="0.022"/>
             <visual>
                 <geometry>

Commit message: fixed Value typo in lidar.xacro

File: urdf/lidar.xacro (robot description, xacro)
@@ -16,5 +16,5 @@
             <xacro:property name="radius" value="0.02"/>
             <xacro:property name="heigth" value="0.01"/>
-            <xacro:property name="mass" value="0.01"/>
+            <xacro:property name="mass" value="0.0134"/>
             <visual>
                 <geometry>
@@ -48,6 +48,6 @@
             <!--radius = 20mm heigth = 1mm-->
             <xacro:property name="radius" value="0.2"/>
-            <xacro:property name="heigth" value="0.1"/>
-            <xacro:property name="mass" value="0.1"/>
+            <xacro:property name="heigth" value="0.01"/>
+            <xacro:property name="mass" value="0.0067"/>
             <visual>
                 <geometry>
